Commit message: create rg2_tipp link

File: resource/model/ur10_rg2_nomimic.urdf (robot description, URDF)
Before this commit: robot ur10, 16 links, 15 joints
Links:
- added link rg2_tipp
Joints:
- added joint rg2_hand-rg2_tipp: type fixed, parent rg2_hand, child rg2_tipp, origin xyz=0.21 0 0 rpy=0 0 0
