Commit message: restructure urdf folder; remove the target key/property and recognize file type automatically; add handleCoppeliaUpload; add sendRos2Cmd and publishMessage for cs_controller

File: Assets/urdf/examples/robots/ur10_rg2/ur10_rg2.urdf (robot description, URDF)
Before this commit: robot ur10, 16 links, 15 joints
Links:
- added link world
- link base: mass 0.001 -> None
- link base_link: mass 0.001 -> None
- link base_link_inertia: geometry collision mesh filename=file:///project-root/Assets/urdf/examples/robots/ur10_rg2/m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; visual mesh filename=file:///project-root/Assets/urdf/examples/robots/ur10_rg2/m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
- link flange: mass 0.001 -> None
- link forearm_link: geometry collision mesh filename=file:///project-root/Assets/urdf/examples/robots/ur10_rg2/m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; visual mesh filename=file:///project-root/Assets/urdf/examples/robots/ur10_rg2/m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
- link ft_frame: mass 0.001 -> None
- link rg2_hand: geometry collision mesh filename=file:///project-root/Assets/urdf/examples/robots/ur10_rg2/m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; visual mesh filename=file:///project-root/Assets/urdf/examples/robots/ur10_rg2/m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
- link rg2_leftfinger: geometry collision mesh filename=file:///project-root/Assets/urdf/examples/robots/ur10_rg2/m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; visual mesh filename=file:///project-root/Assets/urdf/examples/robots/ur10_rg2/m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
- link rg2_rightfinger: geometry collision mesh filename=file:///project-root/Assets/urdf/examples/robots/ur10_rg2/m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; visual mesh filename=file:///project-root/Assets/urdf/examples/robots/ur10_rg2/m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
- link rg2_tipp: mass 0.001 -> None
- link shoulder_link: geometry collision mesh filename=file:///project-root/Assets/urdf/examples/robots/ur10_rg2/m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; visual mesh filename=file:///project-root/Assets/urdf/examples/robots/ur10_rg2/m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
- link tool0: mass 0.001 -> None
- link upper_arm_link: geometry collision mesh filename=file:///project-root/Assets/urdf/examples/robots/ur10_rg2/m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; visual mesh filename=file:///project-root/Assets/urdf/examples/robots/ur10_rg2/m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
- link wrist_1_link: geometry collision mesh filename=file:///project-root/Assets/urdf/examples/robots/ur10_rg2/m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; visual mesh filename=file:///project-root/Assets/urdf/examples/robots/ur10_rg2/m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
- link wrist_2_link: geometry collision mesh filename=file:///project-root/Assets/urdf/examples/robots/ur10_rg2/m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; visual mesh filename=file:///project-root/Assets/urdf/examples/robots/ur10_rg2/m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
- link wrist_3_link: geometry collision mesh filename=file:///project-root/Assets/urdf/examples/robots/ur10_rg2/m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; visual mesh filename=file:///project-root/Assets/urdf/examples/robots/ur10_rg2/m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
Joints:
- added joint base_joint: type fixed, parent world, child base_link, origin xyz=0 0 0 rpy=0 0 0

File: Assets/urdf/examples/robots/ur10_rg2/ur10_rg2_coppelia.urdf (robot description, URDF)
Before this commit: robot ur10, 17 links, 16 joints
Links:
- removed link world
- link base: mass None -> 0.001
- link base_link: mass None -> 0.001
- link base_link_inertia: geometry collision mesh filename=file:///project-root/Assets/urdf/examples/robots/ur10_rg2/m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; visual mesh filename=file:///project-root/Assets/urdf/examples/robots/ur10_rg2/m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
- link flange: mass None -> 0.001
- link forearm_link: geometry collision mesh filename=file:///project-root/Assets/urdf/examples/robots/ur10_rg2/m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; visual mesh filename=file:///project-root/Assets/urdf/examples/robots/ur10_rg2/m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
- link ft_frame: mass None -> 0.001
- link rg2_hand: geometry collision mesh filename=file:///project-root/Assets/urdf/examples/robots/ur10_rg2/m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; visual mesh filename=file:///project-root/Assets/urdf/examples/robots/ur10_rg2/m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
- link rg2_leftfinger: geometry collision mesh filename=file:///project-root/Assets/urdf/examples/robots/ur10_rg2/m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; visual mesh filename=file:///project-root/Assets/urdf/examples/robots/ur10_rg2/m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
- link rg2_rightfinger: geometry collision mesh filename=file:///project-root/Assets/urdf/examples/robots/ur10_rg2/m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; visual mesh filename=file:///project-root/Assets/urdf/examples/robots/ur10_rg2/m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
- link rg2_tipp: mass None -> 0.001
- link shoulder_link: geometry collision mesh filename=file:///project-root/Assets/urdf/examples/robots/ur10_rg2/m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; visual mesh filename=file:///project-root/Assets/urdf/examples/robots/ur10_rg2/m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
- link tool0: mass None -> 0.001
- link upper_arm_link: geometry collision mesh filename=file:///project-root/Assets/urdf/examples/robots/ur10_rg2/m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; visual mesh filename=file:///project-root/Assets/urdf/examples/robots/ur10_rg2/m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
- link wrist_1_link: geometry collision mesh filename=file:///project-root/Assets/urdf/examples/robots/ur10_rg2/m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; visual mesh filename=file:///project-root/Assets/urdf/examples/robots/ur10_rg2/m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
- link wrist_2_link: geometry collision mesh filename=file:///project-root/Assets/urdf/examples/robots/ur10_rg2/m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; visual mesh filename=file:///project-root/Assets/urdf/examples/robots/ur10_rg2/m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
- link wrist_3_link: geometry collision mesh filename=file:///project-root/Assets/urdf/examples/robots/ur10_rg2/m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; visual mesh filename=file:///project-root/Assets/urdf/examples/robots/ur10_rg2/m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
Joints:
- removed joint base_joint
