Commit message: create coppeliasim version ur10 server and urdf; add joint control and joint publish in ur10_rg2_helper; add yaml, moveit scripts and test script for coppeliasim, now robot can be controlled via wot, but gripper apply too much force and can't grab cube

File: Assets/urdf/examples/robots/ur10_rg2/ur10_rg2_coppelia.urdf (robot description, URDF)
Before this commit: robot ur10, 16 links, 15 joints
Joints:
- joint rg2_finger_joint1: limit lower=0.0 upper=1.18 effort=20.0 velocity=2.0 -> lower=0 upper=0.5 effort=0.1 velocity=0.5
- joint rg2_finger_joint2: limit lower=0.0 upper=1.18 effort=20.0 velocity=2.0 -> lower=-0.5 upper=0 effort=0.1 velocity=0.5
